Commit message: Rebase from 'upstream'

File: jsk_2016_01_baxter_apc/robots/baxter.xacro (robot description, xacro)
@@ -1,9 +1,11 @@
 <?xml version="1.0"?>
 <robot xmlns:xacro="http://ros.org/wiki/xacro" name="baxter">
-  <xacro:include filename="$(find jsk_2015_05_baxter_apc)/robots/baxter.xacro" />
+  <xacro:include filename="$(find baxter_description)/urdf/baxter_base/baxter_base.urdf.xacro" />
+  <xacro:include filename="$(find baxter_description)/urdf/pedestal/pedestal.xacro" />
   <!-- Arm Camera -->
   <xacro:include filename="$(find jsk_2016_01_baxter_apc)/robots/right_arm_camera.xacro"/>
   <xacro:include filename="$(find jsk_2016_01_baxter_apc)/robots/left_arm_camera.xacro"/>
-  <!-- Vaccum Gripper-->
+  <!-- Vacuum Gripper -->
+  <xacro:include filename="$(find jsk_2016_01_baxter_apc)/robots/right_vacuum_gripper.xacro"/>
   <xacro:include filename="$(find jsk_2016_01_baxter_apc)/robots/left_vacuum_gripper.xacro"/>
 </robot>

File: jsk_2016_01_baxter_apc/robots/left_arm_camera.xacro (robot description, xacro)
@@ -1,7 +1,7 @@
 <?xml version="1.0"?>
 <robot xmlns:xacro="http://ros.org/wiki/xacro" name="left_arm_camera">
-  <xacro:include filename="$(find softkinetic_camera)/urdf/senz3d.urdf.xacro"/>
-  <xacro:sensor_senz3d name="left_softkinetic_camera" parent="left_wrist">
-    <origin rpy="0 -${M_PI/2} ${M_PI}" xyz="-0.048 0.0 0.10"/>
+  <xacro:include filename="$(find jsk_2016_01_baxter_apc)/robots/softkinetic_camera/senz3d.urdf.xacro"/>
+  <xacro:sensor_senz3d name="left_softkinetic_camera" parent="left_hand">
+    <origin rpy="0 -${M_PI/2} ${M_PI}" xyz="-0.048 0 0.025"/>
   </xacro:sensor_senz3d>
 </robot>

File: jsk_2016_01_baxter_apc/robots/left_vacuum_gripper.xacro (robot description, xacro)
@@ -1,3 +1,50 @@
 <?xml version="1.0"?>
-<robot xmlns:xacro="http://ros.org/wiki/xacro" name="right_vaccum_gripper">
+<robot xmlns:xacro="http://ros.org/wiki/xacro" name="left_vaccum_gripper">
+  <xacro:property name="width" value=".02" />
+  <xacro:property name="width_base" value=".1" />
+  <xacro:property name="width_side2_base" value=".035" />
+  <xacro:property name="bodylen" value=".49" />
+  <xacro:property name="bodylen_base" value=".12" />
+  <xacro:property name="left_wrist_offset_x" value="-0.01" />
+  <link name="left_custom_vacuum_link">
+    <visual>
+      <origin rpy="0 0 1.57" xyz="0 0 -0.07"/>
+      <geometry>
+        <mesh filename="package://jsk_2015_05_baxter_apc/meshes/long1_simple.dae" scale="0.001 0.001 0.001"/>
+      </geometry>
+      <material name="white">
+        <color rgba="1 1 1 1"/>
+      </material>
+    </visual>
+    <collision>
+      <geometry>
+        <cylinder radius="${width}" length="${bodylen}"/>
+      </geometry>
+    </collision>
+  </link>
+  <link name="left_custom_vacuum_link_base">
+    <visual>
+      <geometry>
+        <mesh filename="package://jsk_2015_05_baxter_apc/meshes/light/jigu_long2_left_kari2.dae" scale="0.001 0.001 0.001"/>
+      </geometry>
+      <material name="white">
+        <color rgba="1 1 1 1"/>
+      </material>
+    </visual>
+    <collision>
+      <geometry>
+        <cylinder radius="${width_base}" length="${bodylen_base}"/>
+      </geometry>
+    </collision>
+  </link>
+  <joint name="left_custom_joint" type="fixed">
+    <parent link="left_wrist"/>
+    <child link="left_custom_vacuum_link"/>
+    <origin rpy="0 0 0" xyz="${left_wrist_offset_x} 0 0.19" />
+  </joint>
+  <joint name="left_custom_joint_base" type="fixed">
+    <parent link="left_wrist"/>
+    <child link="left_custom_vacuum_link_base"/>
+    <origin rpy="0 0 1.57" xyz="${left_wrist_offset_x} -0 0.13" />
+  </joint>
 </robot>

File: jsk_2016_01_baxter_apc/robots/right_arm_camera.xacro (robot description, xacro)
@@ -1,7 +1,7 @@
 <?xml version="1.0"?>
 <robot xmlns:xacro="http://ros.org/wiki/xacro" name="right_arm_camera">
-  <xacro:include filename="$(find softkinetic_camera)/urdf/senz3d.urdf.xacro"/>
-  <xacro:sensor_senz3d name="right_softkinetic_camera" parent="right_wrist">
-    <origin rpy="0 -${M_PI/2} ${M_PI}" xyz="-0.048 0.0 0.10"/>
+  <xacro:include filename="$(find jsk_2016_01_baxter_apc)/robots/softkinetic_camera/senz3d.urdf.xacro"/>
+  <xacro:sensor_senz3d name="right_softkinetic_camera" parent="right_hand">
+    <origin rpy="0 -${M_PI/2} ${M_PI}" xyz="-0.048 0 0.025"/>
   </xacro:sensor_senz3d>
 </robot>
