Commit message: Imported upstream version '3.0.0' of 'upstream'

File: jsk_2016_01_baxter_apc/robots/common_constants.xacro (robot description, xacro)
@@ -1,4 +1,4 @@
 <?xml version="1.0"?>
-<robot xmlns:xacro="http://ros.org/wiki/xacro">
+<robot xmlns:xacro="http://www.ros.org/wiki/xacro">
   <xacro:property name="M_PI" value="3.14159265359"/>
 </robot>

File: jsk_2016_01_baxter_apc/robots/left_arm_camera.xacro (robot description, xacro)
@@ -1,4 +1,4 @@
 <?xml version="1.0"?>
-<robot xmlns:xacro="http://ros.org/wiki/xacro" name="left_arm_camera">
+<robot xmlns:xacro="http://www.ros.org/wiki/xacro" name="left_arm_camera">
   <xacro:include filename="$(find jsk_2016_01_baxter_apc)/robots/softkinetic_camera/senz3d.urdf.xacro"/>
   <xacro:sensor_senz3d name="left_softkinetic_camera" parent="left_hand">

File: jsk_2016_01_baxter_apc/robots/left_vacuum_gripper.xacro (robot description, xacro)
@@ -1,5 +1,21 @@
 <?xml version="1.0"?>
-<robot xmlns:xacro="http://ros.org/wiki/xacro" name="left_vaccum_gripper">
+<robot xmlns:xacro="http://www.ros.org/wiki/xacro" name="left_vaccum_gripper">
   <xacro:include filename="$(find jsk_2016_01_baxter_apc)/robots/common_constants.xacro"/>
+  <!-- Gazebo Tags -->
+  <gazebo reference="left_gripper_base">
+    <selfCollide>true</selfCollide>
+    <material>Gazebo/White</material>
+  </gazebo>
+  <gazebo reference="left_gripper_vacuum_pad_base">
+    <selfCollide>true</selfCollide>
+    <material>Gazebo/Grey</material>
+  </gazebo>
+  <gazebo reference="left_gripper_vacuum_pad">
+    <selfCollide>true</selfCollide>
+    <material>Gazebo/Green</material>
+  </gazebo>
+  <gazebo reference="left_gripper_vacuum_pad_joint">
+    <implicitSpringDamper>false</implicitSpringDamper>
+  </gazebo>
   <!--Link bodies-->
   <xacro:property name="rect_tube_l" value="0.285" />
@@ -56,4 +72,9 @@
       </geometry>
     </collision>
+    <inertial>
+      <origin rpy="0 0 0" xyz="0 0 0"/>
+      <mass value="0.3"/>
+      <inertia ixx="0.001" ixy="0" ixz="0" iyy="0.001" iyz="0" izz="0.001"/>
+    </inertial>
   </link>
   <link name="left_gripper_vacuum_pad_base">
@@ -73,4 +94,9 @@
       </geometry>
     </collision>
+    <inertial>
+      <origin rpy="0 0 0" xyz="0 0 0"/>
+      <mass value="0.01"/>
+      <inertia ixx="0.001" ixy="0" ixz="0" iyy="0.001" iyz="0" izz="0.001"/>
+    </inertial>
   </link>
   <link name="left_gripper_vacuum_pad">
@@ -90,4 +116,9 @@
       </geometry>
     </collision>
+    <inertial>
+      <origin rpy="0 0 0" xyz="0 0 0"/>
+      <mass value="0.01"/>
+      <inertia ixx="0.001" ixy="0" ixz="0" iyy="0.001" iyz="0" izz="0.001"/>
+    </inertial>
   </link>
   <joint name="left_gripper_base_fixed" type="fixed">

File: jsk_2016_01_baxter_apc/robots/right_arm_camera.xacro (robot description, xacro)
@@ -1,4 +1,4 @@
 <?xml version="1.0"?>
-<robot xmlns:xacro="http://ros.org/wiki/xacro" name="right_arm_camera">
+<robot xmlns:xacro="http://www.ros.org/wiki/xacro" name="right_arm_camera">
   <xacro:include filename="$(find jsk_2016_01_baxter_apc)/robots/softkinetic_camera/senz3d.urdf.xacro"/>
   <xacro:sensor_senz3d name="right_softkinetic_camera" parent="right_hand">

File: jsk_2016_01_baxter_apc/robots/right_vacuum_gripper.xacro (robot description, xacro)
@@ -1,5 +1,21 @@
 <?xml version="1.0"?>
-<robot xmlns:xacro="http://ros.org/wiki/xacro" name="right_vaccum_gripper">
+<robot xmlns:xacro="http://www.ros.org/wiki/xacro" name="right_vaccum_gripper">
   <xacro:include filename="$(find jsk_2016_01_baxter_apc)/robots/common_constants.xacro"/>
+  <!-- Gazebo Tags -->
+  <gazebo reference="right_gripper_base">
+    <selfCollide>true</selfCollide>
+    <material>Gazebo/White</material>
+  </gazebo>
+  <gazebo reference="right_gripper_vacuum_pad_base">
+    <selfCollide>true</selfCollide>
+    <material>Gazebo/Grey</material>
+  </gazebo>
+  <gazebo reference="right_gripper_vacuum_pad">
+    <selfCollide>true</selfCollide>
+    <material>Gazebo/Green</material>
+  </gazebo>
+  <gazebo reference="right_gripper_vacuum_pad_joint">
+    <implicitSpringDamper>false</implicitSpringDamper>
+  </gazebo>
   <!--Link bodies-->
   <xacro:property name="rect_tube_l" value="0.285" />
@@ -63,4 +79,9 @@
       </geometry>
     </collision>
+    <inertial>
+      <origin rpy="0 0 0" xyz="0 0 0"/>
+      <mass value="0.3"/>
+      <inertia ixx="0.001" ixy="0" ixz="0" iyy="0.001" iyz="0" izz="0.001"/>
+    </inertial>
   </link>
   <link name="right_gripper_vacuum_pad_base">
@@ -87,4 +108,9 @@
       </geometry>
     </collision>
+    <inertial>
+      <origin rpy="0 0 0" xyz="0 0 0"/>
+      <mass value="0.01"/>
+      <inertia ixx="0.001" ixy="0" ixz="0" iyy="0.001" iyz="0" izz="0.001"/>
+    </inertial>
   </link>
   <link name="right_gripper_vacuum_pad">
@@ -111,4 +137,9 @@
       </geometry>
     </collision>
+    <inertial>
+      <origin rpy="0 0 0" xyz="0 0 0"/>
+      <mass value="0.01"/>
+      <inertia ixx="0.001" ixy="0" ixz="0" iyy="0.001" iyz="0" izz="0.001"/>
+    </inertial>
   </link>
   <joint name="right_gripper_base_fixed" type="fixed">
